File: 29f800-adaptor/29f800.sch (KiCad schematic (older format))
At the start: 9 parts, among them J1 Conn_01x02, J2 Conn_01x02, U1 27C400, U2 29F800

Commit message: KiCad 5 libs for 29f800 adapter
Parts:
- C1, C2: footprint Capacitors_SMD:C_0603 -> Capacitor_SMD:C_0603_1608Metric
- J1: footprint Pin_Headers:Pin_Header_Angled_1x02_Pitch2.54mm -> Connector_PinHeader_2.54mm:PinHeader_1x02_P2.54mm_Horizontal
- J2: footprint Pin_Headers:Pin_Header_Straight_1x02_Pitch2.54mm -> Connector_PinHeader_2.54mm:PinHeader_1x02_P2.54mm_Vertical
- R1, R2, R3: footprint Resistors_SMD:R_0603 -> Resistor_SMD:R_0603_1608Metric
- U2: footprint Housings_SSOP:TSOP-I-48_18.4x12mm_Pitch0.5mm -> Package_SO:TSOP-I-48_18.4x12mm_P0.5mm
Changed lines of the file:
@@
 F 0 "U2" H 7000 2200 60  0000 C CNN
 F 1 "29F800" H 7000 -50 60  0000 C CNN
-F 2 "Housings_SSOP:TSOP-I-48_18.4x12mm_Pitch0.5mm" H 7000 2200 60  0001 C CNN
+F 2 "Package_SO:TSOP-I-48_18.4x12mm_P0.5mm" H 7000 2200 60  0001 C CNN
 F 3 "" H 7000 2200 60  0000 C CNN
 	1    7000 2200
@@
 F 0 "R1" H 2320 5596 50  0000 L CNN
 F 1 "10K" H 2320 5505 50  0000 L CNN
-F 2 "Resistors_SMD:R_0603" V 2180 5550 50  0001 C CNN
+F 2 "Resistor_SMD:R_0603_1608Metric" V 2180 5550 50  0001 C CNN
 F 3 "~" H 2250 5550 50  0001 C CNN
 	1    2250 5550
@@
 F 0 "J1" H 1870 5575 50  0000 C CNN
 F 1 "Conn_01x02" H 1870 5666 50  0000 C CNN
-F 2 "Pin_Headers:Pin_Header_Angled_1x02_Pitch2.54mm" H 1950 5900 50  0001 C CNN
+F 2 "Connector_PinHeader_2.54mm:PinHeader_1x02_P2.54mm_Horizontal" H 1950 5900 50  0001 C CNN
 F 3 "~" H 1950 5900 50  0001 C CNN
 	1    1950 5900
@@
 F 0 "J2" H 3370 5575 50  0000 C CNN
 F 1 "Conn_01x02" H 3370 5666 50  0000 C CNN
-F 2 "Pin_Headers:Pin_Header_Straight_1x02_Pitch2.54mm" H 3450 5900 50  0001 C CNN
+F 2 "Connector_PinHeader_2.54mm:PinHeader_1x02_P2.54mm_Vertical" H 3450 5900 50  0001 C CNN
 F 3 "~" H 3450 5900 50  0001 C CNN
 	1    3450 5900
@@
 F 0 "R3" H 3820 5446 50  0000 L CNN
 F 1 "10K" H 3820 5355 50  0000 L CNN
-F 2 "Resistors_SMD:R_0603" V 3680 5400 50  0001 C CNN
+F 2 "Resistor_SMD:R_0603_1608Metric" V 3680 5400 50  0001 C CNN
 F 3 "~" H 3750 5400 50  0001 C CNN
 	1    3750 5400
@@
 F 0 "R2" H 3720 6296 50  0000 L CNN
 F 1 "10K" H 3720 6205 50  0000 L CNN
-F 2 "Resistors_SMD:R_0603" V 3580 6250 50  0001 C CNN
+F 2 "Resistor_SMD:R_0603_1608Metric" V 3580 6250 50  0001 C CNN
 F 3 "~" H 3650 6250 50  0001 C CNN
 	1    3650 6250
@@
 F 0 "C1" H 3365 6296 50  0000 L CNN
 F 1 "0.1uF" H 3365 6205 50  0000 L CNN
-F 2 "Capacitors_SMD:C_0603" H 3288 6100 50  0001 C CNN
+F 2 "Capacitor_SMD:C_0603_1608Metric" H 3288 6100 50  0001 C CNN
 F 3 "~" H 3250 6250 50  0001 C CNN
 	1    3250 6250
@@
 F 0 "C2" H 4915 5696 50  0000 L CNN
 F 1 "0.1uF" H 4915 5605 50  0000 L CNN
-F 2 "Capacitors_SMD:C_0603" H 4838 5500 50  0001 C CNN
+F 2 "Capacitor_SMD:C_0603_1608Metric" H 4838 5500 50  0001 C CNN
 F 3 "~" H 4800 5650 50  0001 C CNN
 	1    4800 5650

Commit message: Added resistors and layout for A500 routing bug
Parts:
- added R4, R5, R6: 0, Resistor_SMD:R_0603_1608Metric, symbol Device:R
- added R7: 10k, Resistor_SMD:R_0603_1608Metric, symbol Device:R
Connections:
- net labels added: P1_1, P1_2, P31_1, P31_2
- net labels removed: P1, P31
- wire segments 107 -> 115
Other:
- note added: "Connect if using A500 V5 \nboard with pin bug"
- note added: "Connect if using boards \nwithout the wrong pin bug \n(Almost all boards)"
Changed lines of the file:
@@
 encoding utf-8
 Sheet 1 1
-Title ""
+Title "29F800 to Amiga kickstart socket Adapter"
 Date ""
 Rev ""
@@
 	7750 4250 8450 4250
 Text Label 2300 2350 0    60   ~ 0
-P1
+P1_1
 Text Label 2300 2450 0    60   ~ 0
 P2
@@
 P_Vss
 Text Label 4600 3250 0    60   ~ 0
-P31
+P31_1
 Text Label 4600 3150 0    60   ~ 0
 P32
@@
 P3
 Text Label 5700 3950 0    60   ~ 0
-P1
+P1_2
 Text Label 5700 4250 0    60   ~ 0
 P4
@@
 P22
 Text Label 8250 2450 0    60   ~ 0
-P31
+P31_2
 Text Label 8250 2550 0    60   ~ 0
 P_Vss
@@
 Wire Wire Line
 	4800 6050 4800 5800
+$Comp
+L Device:R R4
+U 1 1 5BC0BC15
+P 5950 5300
+F 0 "R4" V 5743 5300 50  0000 C CNN
+F 1 "0" V 5834 5300 50  0000 C CNN
+F 2 "Resistor_SMD:R_0603_1608Metric" V 5880 5300 50  0001 C CNN
+F 3 "~" H 5950 5300 50  0001 C CNN
+	1    5950 5300
+	0    1    1    0
+$EndComp
+Text Label 5700 5300 2    50   ~ 0
+P1_1
+Text Label 6200 5300 0    50   ~ 0
+P1_2
+Wire Wire Line
+	5700 5300 5800 5300
+Wire Wire Line
+	6100 5300 6200 5300
+$Comp
+L Device:R R5
+U 1 1 5BC171B2
+P 5950 5650
+F 0 "R5" V 5743 5650 50  0000 C CNN
+F 1 "0" V 5834 5650 50  0000 C CNN
+F 2 "Resistor_SMD:R_0603_1608Metric" V 5880 5650 50  0001 C CNN
+F 3 "~" H 5950 5650 50  0001 C CNN
+	1    5950 5650
+	0    1    1    0
+$EndComp
+Text Label 5700 5650 2    50   ~ 0
+P31_1
+Text Label 6200 5650 0    50   ~ 0
+P31_2
+Wire Wire Line
+	5700 5650 5800 5650
+Wire Wire Line
+	6100 5650 6200 5650
+$Comp
+L Device:R R6
+U 1 1 5BC1B265
+P 5950 6000
+F 0 "R6" V 5743 6000 50  0000 C CNN
+F 1 "0" V 5834 6000 50  0000 C CNN
+F 2 "Resistor_SMD:R_0603_1608Metric" V 5880 6000 50  0001 C CNN
+F 3 "~" H 5950 6000 50  0001 C CNN
+	1    5950 6000
+	0    1    1    0
+$EndComp
+Text Label 5700 6000 2    50   ~ 0
+P31_1
+Text Label 6200 6000 0    50   ~ 0
+P1_2
+Wire Wire Line
+	5700 6000 5800 6000
+Wire Wire Line
+	6100 6000 6200 6000
+$Comp
+L Device:R R7
+U 1 1 5BC1FF61
+P 5950 6350
+F 0 "R7" V 5743 6350 50  0000 C CNN
+F 1 "10k" V 5834 6350 50  0000 C CNN
+F 2 "Resistor_SMD:R_0603_1608Metric" V 5880 6350 50  0001 C CNN
+F 3 "~" H 5950 6350 50  0001 C CNN
+	1    5950 6350
+	0    1    1    0
+$EndComp
+Text Label 6200 6350 0    50   ~ 0
+P31_2
+Wire Wire Line
+	5700 6350 5800 6350
+Wire Wire Line
+	6100 6350 6200 6350
+$Comp
+L power:VCC #PWR08
+U 1 1 5BC24639
+P 5700 6350
+F 0 "#PWR08" H 5700 6200 50  0001 C CNN
+F 1 "VCC" H 5717 6523 50  0000 C CNN
+F 2 "" H 5700 6350 50  0001 C CNN
+F 3 "" H 5700 6350 50  0001 C CNN
+	1    5700 6350
+	1    0    0    -1
+$EndComp
+Wire Notes Line
+	7650 6450 5400 6450
+Wire Notes Line
+	5400 5750 7650 5750
+Text Notes 6600 6150 0    50   ~ 0
+Connect if using A500 V5 \nboard with pin bug
+Wire Notes Line
+	5400 5000 7650 5000
+Wire Notes Line
+	5400 5000 5400 6450
+Wire Notes Line
+	7650 5000 7650 6450
+Text Notes 6500 5450 0    50   ~ 0
+Connect if using boards \nwithout the wrong pin bug \n(Almost all boards)
 $EndSCHEMATC
