File: 29f800-prog/29f800-prog.sch (KiCad schematic (older format))
At the start: 3 parts

Commit message: Programming adapter
Parts:
- added J2: Conn_01x04, Connector_PinHeader_2.54mm:PinHeader_1x04_P2.54mm_Vertical, symbol Connector_Generic:Conn_01x04
- added U2: 29f800_48p, symbol FF:29f800_48p
- J1, J3: renamed from J?; footprint (none) -> Connector_PinHeader_2.54mm:PinHeader_2x12_P2.54mm_Vertical
- U1: renamed from U?; footprint (none) -> Package_DIP:DIP-40_W15.24mm_Socket
Connections:
- net labels added: P1, P11, P12, P15, P16, P17, P18, P19, P2, P20, P21, P22, P23, P24, P28, P29, P3, P30, P31, P32, P33, P34, P35, P36, P37, P38, P39, P4, P40, P41, P42, P43, P44, P45, P46, P47, P48, P5, P6, P7, P8
Changed lines of the file:
@@
 EESchema Schematic File Version 4
+LIBS:29f800-prog-cache
 EELAYER 26 0
 EELAYER END
@@
 $EndDescr
 $Comp
-L FF:AmigaSocket U?
+L FF:AmigaSocket U1
 U 1 1 5BC0912E
 P 5750 2500
-F 0 "U?" H 5750 2637 60  0000 C CNN
+F 0 "U1" H 5750 2637 60  0000 C CNN
 F 1 "AmigaSocket" H 5750 2531 60  0000 C CNN
-F 2 "" H 5750 2500 60  0000 C CNN
+F 2 "Package_DIP:DIP-40_W15.24mm_Socket" H 5750 2500 60  0000 C CNN
 F 3 "" H 5750 2500 60  0000 C CNN
 	1    5750 2500
@@
 $EndComp
 $Comp
-L Connector_Generic:Conn_02x12_Odd_Even J?
+L Connector_Generic:Conn_02x12_Odd_Even J1
 U 1 1 5BC0931E
 P 2950 3500
-F 0 "J?" H 3000 4217 50  0000 C CNN
+F 0 "J1" H 3000 4217 50  0000 C CNN
 F 1 "Conn_02x12_Odd_Even" H 3000 4126 50  0000 C CNN
-F 2 "" H 2950 3500 50  0001 C CNN
+F 2 "Connector_PinHeader_2.54mm:PinHeader_2x12_P2.54mm_Vertical" H 2950 3500 50  0001 C CNN
 F 3 "~" H 2950 3500 50  0001 C CNN
 	1    2950 3500
@@
 $EndComp
 $Comp
-L Connector_Generic:Conn_02x12_Odd_Even J?
+L Connector_Generic:Conn_02x12_Odd_Even J3
 U 1 1 5BC09420
 P 8550 3500
-F 0 "J?" H 8600 4217 50  0000 C CNN
+F 0 "J3" H 8600 4217 50  0000 C CNN
 F 1 "Conn_02x12_Odd_Even" H 8600 4126 50  0000 C CNN
-F 2 "" H 8550 3500 50  0001 C CNN
+F 2 "Connector_PinHeader_2.54mm:PinHeader_2x12_P2.54mm_Vertical" H 8550 3500 50  0001 C CNN
 F 3 "~" H 8550 3500 50  0001 C CNN
 	1    8550 3500
@@
 Text Label 8850 4000 0    50   ~ 0
 P27
+Text Label 8350 4000 2    50   ~ 0
+P28
+Text Label 8350 3900 2    50   ~ 0
+P30
+Text Label 8350 3800 2    50   ~ 0
+P32
+Text Label 8350 3700 2    50   ~ 0
+P34
+Text Label 8350 3600 2    50   ~ 0
+P36
+Text Label 8350 3500 2    50   ~ 0
+P38
+Text Label 8350 3400 2    50   ~ 0
+P40
+Text Label 8350 3300 2    50   ~ 0
+P42
+Text Label 8350 3200 2    50   ~ 0
+P44
+Text Label 8350 3100 2    50   ~ 0
+P46
+Text Label 8350 3000 2    50   ~ 0
+P48
+Text Label 8850 3900 0    50   ~ 0
+P29
+Text Label 8850 3800 0    50   ~ 0
+P31
+Text Label 8850 3700 0    50   ~ 0
+P33
+Text Label 8850 3600 0    50   ~ 0
+P35
+Text Label 8850 3500 0    50   ~ 0
+P37
+Text Label 8850 3400 0    50   ~ 0
+P39
+Text Label 8850 3300 0    50   ~ 0
+P41
+Text Label 8850 3200 0    50   ~ 0
+P43
+Text Label 8850 3100 0    50   ~ 0
+P45
+Text Label 8850 3000 0    50   ~ 0
+P47
+$Comp
+L FF:29f800_48p U2
+U 1 1 5BC2FE6C
+P 5800 4850
+F 0 "U2" H 5800 4987 60  0000 C CNN
+F 1 "29f800_48p" H 5800 4881 60  0000 C CNN
+F 2 "" H 5800 4850 60  0000 C CNN
+F 3 "" H 5800 4850 60  0000 C CNN
+	1    5800 4850
+	1    0    0    -1
+$EndComp
+Text Label 5000 2650 2    50   ~ 0
+P17
+Text Label 5000 2750 2    50   ~ 0
+P18
+Text Label 5000 2850 2    50   ~ 0
+P19
+Text Label 5000 2950 2    50   ~ 0
+P20
+Text Label 5000 3050 2    50   ~ 0
+P21
+Text Label 5000 3150 2    50   ~ 0
+P22
+Text Label 5000 3250 2    50   ~ 0
+P23
+Text Label 5000 3350 2    50   ~ 0
+P24
+Text Label 5000 3450 2    50   ~ 0
+P25
+Text Label 5000 3650 2    50   ~ 0
+P27
+Text Label 5000 3850 2    50   ~ 0
+P29
+Text Label 5000 3950 2    50   ~ 0
+P30
+Text Label 5000 4050 2    50   ~ 0
+P31
+Text Label 5000 4150 2    50   ~ 0
+P32
+Text Label 5000 4250 2    50   ~ 0
+P33
+Text Label 5000 4350 2    50   ~ 0
+P34
+Text Label 5000 4450 2    50   ~ 0
+P35
+Text Label 5000 4550 2    50   ~ 0
+P36
+Text Label 6500 2650 0    50   ~ 0
+P8
+Text Label 6500 2750 0    50   ~ 0
+P7
+Text Label 6500 2850 0    50   ~ 0
+P6
+Text Label 6500 2950 0    50   ~ 0
+P5
+Text Label 6500 3050 0    50   ~ 0
+P4
+Text Label 6500 3150 0    50   ~ 0
+P3
+Text Label 6500 3250 0    50   ~ 0
+P2
+Text Label 6500 3350 0    50   ~ 0
+P1
+Text Label 6500 3450 0    50   ~ 0
+P48
+Text Label 6500 3550 0    50   ~ 0
+P47
+Text Label 6500 3650 0    50   ~ 0
+P46
+Text Label 6500 3750 0    50   ~ 0
+P45
+Text Label 6500 3850 0    50   ~ 0
+P44
+Text Label 6500 3950 0    50   ~ 0
+P43
+Text Label 6500 4050 0    50   ~ 0
+P42
+Text Label 6500 4150 0    50   ~ 0
+P41
+Text Label 6500 4250 0    50   ~ 0
+P40
+Text Label 6500 4350 0    50   ~ 0
+P39
+Text Label 6500 4450 0    50   ~ 0
+P38
+Text Label 6500 4550 0    50   ~ 0
+P37
+Text Label 2750 3000 2    50   ~ 0
+P1
+Text Label 2750 3100 2    50   ~ 0
+P3
+Text Label 2750 3200 2    50   ~ 0
+P5
+Text Label 2750 3300 2    50   ~ 0
+P7
+Text Label 2750 3500 2    50   ~ 0
+P11
+Text Label 2750 3700 2    50   ~ 0
+P15
+Text Label 2750 3800 2    50   ~ 0
+P17
+Text Label 2750 3900 2    50   ~ 0
+P19
+Text Label 2750 4000 2    50   ~ 0
+P21
+Text Label 2750 4100 2    50   ~ 0
+P23
+Text Label 3250 3000 0    50   ~ 0
+P2
+Text Label 3250 3100 0    50   ~ 0
+P4
+Text Label 3250 3200 0    50   ~ 0
+P6
+Text Label 3250 3300 0    50   ~ 0
+P8
+Text Label 3250 3500 0    50   ~ 0
+P12
+Text Label 3250 3700 0    50   ~ 0
+P16
+Text Label 3250 3800 0    50   ~ 0
+P18
+Text Label 3250 3900 0    50   ~ 0
+P20
+Text Label 3250 4000 0    50   ~ 0
+P22
+Text Label 3250 4100 0    50   ~ 0
+P24
+$Comp
+L Connector_Generic:Conn_01x04 J2
+U 1 1 5BC31050
+P 4050 4700
+F 0 "J2" H 4130 4692 50  0000 L CNN
+F 1 "Conn_01x04" H 4130 4601 50  0000 L CNN
+F 2 "Connector_PinHeader_2.54mm:PinHeader_1x04_P2.54mm_Vertical" H 4050 4700 50  0001 C CNN
+F 3 "~" H 4050 4700 50  0001 C CNN
+	1    4050 4700
+	1    0    0    -1
+$EndComp
+Text Label 3850 4600 2    50   ~ 0
+P11
+Text Label 3850 4700 2    50   ~ 0
+P12
+Text Label 3850 4800 2    50   ~ 0
+P15
+Text Label 3850 4900 2    50   ~ 0
+P16
+Text Label 5000 3550 2    50   ~ 0
+P26
+Text Label 5000 3750 2    50   ~ 0
+P28
 $EndSCHEMATC
